Commit message: Editing gazebo.launch.py file

File: ros2_ws/install/amr_description/share/amr_description/urdf/amr.xacro (robot description, xacro)
@@ -1,243 +1 @@
-<?xml version='1.0' encoding='utf-8'?>
-<robot name="amr" xmlns:xacro="http://www.ros.org/wiki/xacro">
-  <!-- Include materials -->
-  <xacro:include filename="$(find amr_description)/urdf/materials.xacro"/>
-  <!-- Include gazebo -->
-  <xacro:include filename="$(find amr_description)/urdf/gazebo.xacro"/>
-<!--Base Link-->
-    <link name="base_link">
-        <inertial>
-            <origin xyz="-0.005375575226534499 -5.49485313734377e-17 -0.04376770691964268" rpy="0.0 0.0 0.0" />
-            <mass value="1330.496380521211" />
-            <inertia ixx="64.9238607790594" iyy="107.9255209958365" izz="158.45361638099502" ixy="-1.8676558262176537e-13" iyz="-3.189242911227797e-14" ixz="0.5575992010593869" />
-        </inertial>
-        <visual name="base_link_visual">
-            <origin xyz="0.0 0.0 0.0" rpy="0.0 0.0 0.0" />
-            <geometry>
-                <mesh filename="package://amr_description/meshes/base_link.stl" scale="0.001 0.001 0.001" />
-            </geometry>
-            <material name="base_link"/>
-        </visual>
-        <collision name="base_link_collision">
-            <origin xyz="0.0 0.0 0.0" rpy="0.0 0.0 0.0" />
-            <geometry>
-                <mesh filename="package://amr_description/meshes/base_link.stl" scale="0.001 0.001 0.001" />
-            </geometry>
-        </collision>
-    </link>
-<!--Wheels-->
-    <link name="f_wheel_r">
-        <inertial>
-            <origin xyz="0.0 3.552713678800501e-17 0.07500000000000007" rpy="0.0 -0.0 0.0" />
-            <mass value="27.390760948486008" />
-            <inertia ixx="0.47933831659850945" iyy="0.4793383165984846" izz="0.8559612796401739" ixy="3.3306690738754696e-16" iyz="-5.551115123125783e-16" ixz="1.7763568394002505e-15" />
-        </inertial>
-        <visual name="f_wheel_r_visual">
-            <origin xyz="-0.4 0.065 -0.425" rpy="-1.5707963267948966 -0.0 0.0" />
-            <geometry>
-                <mesh filename="package://amr_description/meshes/f_wheel_r.stl" scale="0.001 0.001 0.001" />
-            </geometry>
-            <material name="Wheels"/>
-        </visual>
-        <collision name="f_wheel_r_collision">
-            <origin xyz="-0.4 0.065 -0.425" rpy="-1.5707963267948966 -0.0 0.0" />
-            <geometry>
-                <mesh filename="package://amr_description/meshes/f_wheel_r.stl" scale="0.001 0.001 0.001" />
-            </geometry>
-        </collision>
-    </link>
-    <link name="f_wheel_l">
-        <inertial>
-            <origin xyz="0.0 -3.552713678800501e-17 0.075" rpy="0.0 -0.0 0.0" />
-            <mass value="27.390760948486008" />
-            <inertia ixx="0.4793383165985121" iyy="0.47933831659848636" izz="0.8559612796401739" ixy="-3.3306690738754696e-16" iyz="3.3306690738754696e-16" ixz="0.0" />
-        </inertial>
-        <visual name="f_wheel_l_visual">
-            <origin xyz="-0.4 -0.065 -0.425" rpy="1.5707963267948966 -0.0 0.0" />
-            <geometry>
-                <mesh filename="package://amr_description/meshes/f_wheel_l.stl" scale="0.001 0.001 0.001" />
-            </geometry>
-            <material name="Wheels"/>
-        </visual>
-        <collision name="f_wheel_l_collision">
-            <origin xyz="-0.4 -0.065 -0.425" rpy="1.5707963267948966 -0.0 0.0" />
-            <geometry>
-                <mesh filename="package://amr_description/meshes/f_wheel_l.stl" scale="0.001 0.001 0.001" />
-            </geometry>
-        </collision>
-    </link>
-    <link name="b_wheel_r">
-        <inertial>
-            <origin xyz="0.0 3.552713678800501e-17 0.07500000000000007" rpy="0.0 -0.0 0.0" />
-            <mass value="27.390760948486008" />
-            <inertia ixx="0.47933831659850945" iyy="0.4793383165984846" izz="0.8559612796401739" ixy="3.3306690738754696e-16" iyz="-5.551115123125783e-16" ixz="-2.6645352591003757e-15" />
-        </inertial>
-        <visual name="b_wheel_r_visual">
-            <origin xyz="0.4 0.065 -0.425" rpy="-1.5707963267948966 -0.0 0.0" />
-            <geometry>
-                <mesh filename="package://amr_description/meshes/b_wheel_r.stl" scale="0.001 0.001 0.001" />
-            </geometry>
-            <material name="Wheels"/>
-        </visual>
-        <collision name="b_wheel_r_collision">
-            <origin xyz="0.4 0.065 -0.425" rpy="-1.5707963267948966 -0.0 0.0" />
-            <geometry>
-                <mesh filename="package://amr_description/meshes/b_wheel_r.stl" scale="0.001 0.001 0.001" />
-            </geometry>
-        </collision>
-    </link>
-    <link name="b_wheel_l">
-        <inertial>
-            <origin xyz="0.0 -3.552713678800501e-17 0.075" rpy="0.0 -0.0 0.0" />
-            <mass value="27.390760948486008" />
-            <inertia ixx="0.4793383165985121" iyy="0.47933831659848636" izz="0.8559612796401739" ixy="-3.3306690738754696e-16" iyz="3.3306690738754696e-16" ixz="0.0" />
-        </inertial>
-        <visual name="b_wheel_l_visual">
-            <origin xyz="0.4 -0.065 -0.425" rpy="1.5707963267948966 -0.0 0.0" />
-            <geometry>
-                <mesh filename="package://amr_description/meshes/b_wheel_l.stl" scale="0.001 0.001 0.001" />
-            </geometry>
-            <material name="Wheels"/>
-        </visual>
-        <collision name="b_wheel_l_collision">
-            <origin xyz="0.4 -0.065 -0.425" rpy="1.5707963267948966 -0.0 0.0" />
-            <geometry>
-                <mesh filename="package://amr_description/meshes/b_wheel_l.stl" scale="0.001 0.001 0.001" />
-            </geometry>
-        </collision>
-    </link>
-<!--Camera link-->
-    <link name="camera_link">
-        <inertial>
-            <origin xyz="0.00021147401675925437 1.1102230246251566e-18 0.05000000000000004" rpy="0.0 -0.0 0.0" />
-            <mass value="21.86537558266994" />
-            <inertia ixx="0.16402649642970402" iyy="0.03558843780421217" izz="0.16574154808891284" ixy="2.4125911295413974e-14" iyz="4.5693013817071915e-17" ixz="2.220446049250313e-16" />
-        </inertial>
-        <visual name="camera_link_visual">
-            <origin xyz="-0.19166700333333336 1.1102230246251566e-18 -0.23500000000000001" rpy="0.0 -0.0 0.0" />
-            <geometry>
-                <mesh filename="package://amr_description/meshes/camera_link.stl" scale="0.001 0.001 0.001" />
-            </geometry>
-            <material name="camera_link"/>
-        </visual>
-        <collision name="camera_link_collision">
-            <origin xyz="-0.19166700333333336 1.1102230246251566e-18 -0.23500000000000001" rpy="0.0 -0.0 0.0" />
-            <geometry>
-                <mesh filename="package://amr_description/meshes/camera_link.stl" scale="0.001 0.001 0.001" />
-            </geometry>
-        </collision>
-    </link>
-<!--Lidar link-->
-    <link name="lidar_link">
-        <inertial>
-            <origin xyz="0.0 -1.8528073920390496e-17 0.04" rpy="0.0 -0.0 0.0" />
-            <mass value="30.826877913349836" />
-            <inertia ixx="0.13685849340280387" iyy="0.1368584934028112" izz="0.24083498369804202" ixy="1.8277205526828766e-16" iyz="3.1413946999236946e-17" ixz="0.0" />
-        </inertial>
-        <visual name="lidar_link_visual">
-            <origin xyz="0.0 0.0 -0.185" rpy="3.141592653589793 -0.0 0.0" />
-            <geometry>
-                <mesh filename="package://amr_description/meshes/lidar_link.stl" scale="0.001 0.001 0.001" />
-            </geometry>
-            <material name="lidar_link"/>
-        </visual>
-        <collision name="lidar_link_collision">
-            <origin xyz="0.0 0.0 -0.185" rpy="3.141592653589793 -0.0 0.0" />
-            <geometry>
-                <mesh filename="package://amr_description/meshes/lidar_link.stl" scale="0.001 0.001 0.001" />
-            </geometry>
-        </collision>
-    </link>
-<!--Joints-->
-    <joint name="f_wheel_r_revolute" type="continuous">
-        <origin xyz="0.4 -0.425 -0.065" rpy="1.5707963267948966 -0.0 0.0" />
-        <parent link="base_link" />
-        <child link="f_wheel_r" />
-        <axis xyz="0.0 0.0 1.0" />
-    </joint>
-    <joint name="f_wheel_l_revolute" type="continuous">
-        <origin xyz="0.4 0.425 -0.065" rpy="-1.5707963267948966 -0.0 0.0" />
-        <parent link="base_link" />
-        <child link="f_wheel_l" />
-        <axis xyz="0.0 0.0 1.0" />
-    </joint>
-    <joint name="b_wheel_l_revolute" type="continuous">
-        <origin xyz="-0.4 0.425 -0.065" rpy="-1.5707963267948966 -0.0 0.0" />
-        <parent link="base_link" />
-        <child link="b_wheel_l" />
-        <axis xyz="0.0 0.0 1.0" />
-    </joint>
-    <joint name="b_wheel_r_revolute" type="continuous">
-        <origin xyz="-0.4 -0.425 -0.065" rpy="1.5707963267948966 -0.0 0.0" />
-        <parent link="base_link" />
-        <child link="b_wheel_r" />
-        <axis xyz="0.0 0.0 1.0" />
-    </joint>
-    <joint name="camera_rotation" type="continuous">
-        <origin xyz="0.19166667 0.0 0.23500000000000001" rpy="0.0 -0.0 0.0" />
-        <parent link="base_link" />
-        <child link="camera_link" />
-        <axis xyz="0.0 0.0 1.0" />
-        <limit lower="-1.5707963267948966" upper="1.5707963267948966" effort="100" velocity="1.0"/>
-    </joint>
-    <joint name="lidar_rotation" type="continuous">
-        <origin xyz="0.0 0.0 -0.185" rpy="3.141592653589793 -0.0 0.0" />
-        <parent link="base_link" />
-        <child link="lidar_link" />
-        <axis xyz="0.0 0.0 1.0" />
-    </joint>
-    <!-- Camera Sensor Plugin -->
-        <gazebo reference="camera_link">
-            <sensor name="camera_sensor" type="camera">
-                <topic>camera/image_raw</topic>
-                <update_rate>30.0</update_rate>
-                <camera>
-                    <horizontal_fov>1.047</horizontal_fov>
-                    <image>
-                        <width>640</width>
-                        <height>480</height>
-                        <format>R8G8B8</format>
-                    </image>
-                    <clip>
-                        <near>0.1</near>
-                        <far>100.0</far>
-                    </clip>
-                </camera>
-                <plugin name="camera_controller" filename="libgazebo_ros_camera.so">
-                    <ros>
-                        <namespace>/camera</namespace>
-                    </ros>
-                    <frame_name>camera_link</frame_name>
-                </plugin>
-            </sensor>
-        </gazebo>
-    <!-- LiDAR Sensor Plugin -->
-        <gazebo reference="lidar_link">
-            <sensor name="lidar_sensor" type="ray">
-                <topic>scan</topic>
-                <update_rate>10.0</update_rate>
-                <ray>
-                    <scan>
-                        <horizontal>
-                            <samples>720</samples>
-                            <resolution>1</resolution>
-                            <min_angle>-3.14159</min_angle>
-                            <max_angle>3.14159</max_angle>
-                        </horizontal>
-                    </scan>
-                    <range>
-                        <min>0.12</min>
-                        <max>12.0</max>
-                        <resolution>0.01</resolution>
-                    </range>
-                </ray>
-                <plugin name="laser_controller" filename="libgazebo_ros_ray_sensor.so">
-                    <ros>
-                        <remapping>~/out:=scan</remapping>
-                    </ros>
-                    <output_type>sensor_msgs/LaserScan</output_type>
-                    <frame_name>lidar_link</frame_name>
-                </plugin>
-            </sensor>
-        </gazebo>
-</robot>
+/home/sam/amr-simulation/ros2_ws/src/amr_description/urdf/amr.xacro

File: ros2_ws/install/amr_description/share/amr_description/urdf/gazebo.xacro (robot description, xacro)
@@ -1,74 +1 @@
-<?xml version="1.0"?>
-<robot xmlns:xacro="http://www.ros.org/wiki/xacro">
-    <!-- ================= BASE LINK ================= -->
-    <gazebo reference="base_link">
-        <material>Gazebo/Orange</material>
-        <mu1>1.0</mu1>
-        <mu2>1.0</mu2>
-        <kp>1000000.0</kp>
-        <kd>100.0</kd>
-    </gazebo>
-    <!-- ================= RIGHT WHEEL 1 ================= -->
-    <gazebo reference="r_wheel_link_1">
-        <material>Gazebo/Black</material>
-        <mu1>2.0</mu1>
-        <mu2>2.0</mu2>
-        <kp>1000000.0</kp>
-        <kd>100.0</kd>
-        <fdir1>1 0 0</fdir1>
-    </gazebo>
-    <!-- ================= RIGHT WHEEL 2 ================= -->
-    <gazebo reference="r_wheel_link_2">
-        <material>Gazebo/Black</material>
-        <mu1>2.0</mu1>
-        <mu2>2.0</mu2>
-        <kp>1000000.0</kp>
-        <kd>100.0</kd>
-        <fdir1>1 0 0</fdir1>
-    </gazebo>
-    <!-- ================= LEFT WHEEL 1 ================= -->
-    <gazebo reference="l_wheel_link_1">
-        <material>Gazebo/Black</material>
-        <mu1>2.0</mu1>
-        <mu2>2.0</mu2>
-        <kp>1000000.0</kp>
-        <kd>100.0</kd>
-        <fdir1>1 0 0</fdir1>
-    </gazebo>
-    <!-- ================= LEFT WHEEL 2 ================= -->
-    <gazebo reference="l_wheel_link_2">
-        <material>Gazebo/Black</material>
-        <mu1>2.0</mu1>
-        <mu2>2.0</mu2>
-        <kp>1000000.0</kp>
-        <kd>100.0</kd>
-        <fdir1>1 0 0</fdir1>
-    </gazebo>
-    <!-- ================= DIFFERENTIAL DRIVE ================= -->
-    <gazebo>
-        <plugin name="diff_drive_controller"
-                filename="libgazebo_ros_diff_drive.so">
-            <ros>
-                <namespace>/</namespace>
-            </ros>
-            <update_rate>50</update_rate>
-            <!-- LEFT SIDE -->
-            <left_joint>l_wheel_joint_1</left_joint>
-            <left_joint>l_wheel_joint_2</left_joint>
-            <!-- RIGHT SIDE -->
-            <right_joint>r_wheel_joint_1</right_joint>
-            <right_joint>r_wheel_joint_2</right_joint>
-            <wheel_separation>0.32</wheel_separation>
-            <wheel_diameter>0.10</wheel_diameter>
-            <max_wheel_torque>20</max_wheel_torque>
-            <max_wheel_acceleration>10.0</max_wheel_acceleration>
-            <publish_odom>true</publish_odom>
-            <publish_odom_tf>true</publish_odom_tf>
-            <publish_wheel_tf>true</publish_wheel_tf>
-            <odometry_frame>odom</odometry_frame>
-            <robot_base_frame>base_link</robot_base_frame>
-            <command_topic>cmd_vel</command_topic>
-            <odometry_topic>odom</odometry_topic>
-        </plugin>
-    </gazebo>
-</robot>
+/home/sam/amr-simulation/ros2_ws/src/amr_description/urdf/gazebo.xacro

File: ros2_ws/install/amr_description/share/amr_description/urdf/materials.xacro (robot description, xacro)
@@ -1,16 +1 @@
-<?xml version="1.0"?>
-<robot xmlns:xacro="http://www.ros.org/wiki/xacro">
-    <!-- ================= COLORS ================= -->
-    <material name="Wheels">
-        <color rgba="0.05 0.05 0.05 1"/>
-    </material>
-    <material name="base_link">
-        <color rgba="0.85 0.55 0.1 1"/>
-    </material>
-    <material name="camera_link">
-        <color rgba="1 0 0 1"/>
-    </material>
-    <material name="lidar_link">
-        <color rgba="0 1 0 1"/>
-    </material>
-</robot>
+/home/sam/amr-simulation/ros2_ws/src/amr_description/urdf/materials.xacro

File: ros2_ws/src/amr_description/urdf/amr.urdf (robot description, URDF)
Before this commit: robot amr, 7 links, 6 joints
Links:
- link b_wheel_l: mass 27.390760948486008 -> 1.31279161885651; geometry collision mesh filename=package://amr_description/meshes/b_wheel_l.stl scale=0.001 0.001 0.001; visual mesh filename=package://amr_description/meshes/b_wheel_l.stl scale=0.001 0.001 0.001
- link b_wheel_r: mass 27.390760948486008 -> 1.31279161885651; geometry collision mesh filename=package://amr_description/meshes/b_wheel_r.stl scale=0.001 0.001 0.001; visual mesh filename=package://amr_description/meshes/b_wheel_r.stl scale=0.001 0.001 0.001
- link base_link: mass 1330.496380521211 -> 0.9360217886690454; geometry collision mesh filename=package://amr_description/meshes/base_link.stl scale=0.001 0.001 0.001; visual mesh filename=package://amr_description/meshes/base_link.stl scale=0.001 0.001 0.001
- link camera_link: mass 21.86537558266994 -> 0.03705472598311712; geometry collision mesh filename=package://amr_description/meshes/camera_link.stl scale=0.001 0.001 0.001; visual mesh filename=package://amr_description/meshes/camera_link.stl scale=0.001 0.001 0.001
- link f_wheel_l: mass 27.390760948486008 -> 1.3127916188565103; geometry collision mesh filename=package://amr_description/meshes/f_wheel_l.stl scale=0.001 0.001 0.001; visual mesh filename=package://amr_description/meshes/f_wheel_l.stl scale=0.001 0.001 0.001
- link f_wheel_r: mass 27.390760948486008 -> 1.3127916188565099; geometry collision mesh filename=package://amr_description/meshes/f_wheel_r.stl scale=0.001 0.001 0.001; visual mesh filename=package://amr_description/meshes/f_wheel_r.stl scale=0.001 0.001 0.001
- link lidar_link: mass 30.826877913349836 -> 0.33441151294791577; geometry collision mesh filename=package://amr_description/meshes/lidar_link.stl scale=0.001 0.001 0.001; visual mesh filename=package://amr_description/meshes/lidar_link.stl scale=0.001 0.001 0.001
Joints:
- removed joint base_link_b_wheel_l_revolute
- removed joint base_link_b_wheel_r_revolute
- removed joint base_link_camera_rotation
- removed joint base_link_f_wheel_l_revolute
- removed joint base_link_f_wheel_r_revolute
- removed joint base_link_lidar_rotation
- added joint b_wheel_l_revolute: type continuous, parent base_link, child b_wheel_l, origin xyz=-0.15 0.15937500000000002 -0.0025 rpy=-1.5707963267948966 -0.0 0.0, axis 0.0 0.0 1.0
- added joint b_wheel_r_revolute: type continuous, parent base_link, child b_wheel_r, origin xyz=-0.15 -0.15937500000000002 -0.0025 rpy=1.5707963267948966 -0.0 0.0, axis 0.0 0.0 1.0
- added joint camera_rotation: type revolute, parent base_link, child camera_link, origin xyz=0.07187500000000001 0.0 0.11 rpy=0.0 -0.0 0.0, axis 0.0 0.0 1.0, limit lower=-1.5707963267948966 upper=1.5707963267948966 effort=100 velocity=1.0
- added joint f_wheel_l_revolute: type continuous, parent base_link, child f_wheel_l, origin xyz=0.15 0.15937500000000002 -0.0025 rpy=-1.5707963267948966 -0.0 0.0, axis 0.0 0.0 1.0
- added joint f_wheel_r_revolute: type continuous, parent base_link, child f_wheel_r, origin xyz=0.15 -0.15937500000000002 -0.0025 rpy=1.5707963267948966 -0.0 0.0, axis 0.0 0.0 1.0
- added joint lidar_rotation: type continuous, parent base_link, child lidar_link, origin xyz=0.0 0.0 -0.0475 rpy=3.141592653589793 -0.0 0.0, axis 0.0 0.0 1.0
