Commit message: Editing gazebo.launch.py file

File: ros2_ws/src/amr_description/urdf/amr.xacro (robot description, xacro)
@@ -8,7 +8,7 @@
     <link name="base_link">
         <inertial>
-            <origin xyz="-0.005375575226534499 -5.49485313734377e-17 -0.04376770691964268" rpy="0.0 0.0 0.0" />
-            <mass value="1330.496380521211" />
-            <inertia ixx="64.9238607790594" iyy="107.9255209958365" izz="158.45361638099502" ixy="-1.8676558262176537e-13" iyz="-3.189242911227797e-14" ixz="0.5575992010593869" />
+            <origin xyz="-0.004351267108603693 -2.5010522091502847e-16 0.008281830778488642" rpy="0.0 0.0 0.0" />
+            <mass value="0.9360217886690454" />
+            <inertia ixx="0.009459041504582138" iyy="0.013956118845845198" izz="0.020474384137866695" ixy="5.096082182149493e-17" iyz="6.777214071700385e-17" ixz="0.00014505282040201085" />
         </inertial>
         <visual name="base_link_visual">
@@ -29,10 +29,10 @@
     <link name="f_wheel_r">
         <inertial>
-            <origin xyz="0.0 3.552713678800501e-17 0.07500000000000007" rpy="0.0 -0.0 0.0" />
-            <mass value="27.390760948486008" />
-            <inertia ixx="0.47933831659850945" iyy="0.4793383165984846" izz="0.8559612796401739" ixy="3.3306690738754696e-16" iyz="-5.551115123125783e-16" ixz="1.7763568394002505e-15" />
+            <origin xyz="-1.7763568394002505e-17 -4.440892098500626e-18 0.026235066114433145" rpy="0.0 -0.0 0.0" />
+            <mass value="1.3127916188565099" />
+            <inertia ixx="0.003348709408788453" iyy="0.0033487094087883557" izz="0.0060726776588351" ixy="-1.6263032587282567e-18" iyz="2.710505431213761e-18" ixz="0.0" />
         </inertial>
         <visual name="f_wheel_r_visual">
-            <origin xyz="-0.4 0.065 -0.425" rpy="-1.5707963267948966 -0.0 0.0" />
+            <origin xyz="-0.15 0.0025 -0.15937500000000002" rpy="-1.5707963267948966 -0.0 0.0" />
             <geometry>
                 <mesh filename="package://amr_description/meshes/f_wheel_r.stl" scale="0.001 0.001 0.001" />
@@ -41,5 +41,5 @@
         </visual>
         <collision name="f_wheel_r_collision">
-            <origin xyz="-0.4 0.065 -0.425" rpy="-1.5707963267948966 -0.0 0.0" />
+            <origin xyz="-0.15 0.0025 -0.15937500000000002" rpy="-1.5707963267948966 -0.0 0.0" />
             <geometry>
                 <mesh filename="package://amr_description/meshes/f_wheel_r.stl" scale="0.001 0.001 0.001" />
@@ -49,10 +49,10 @@
     <link name="f_wheel_l">
         <inertial>
-            <origin xyz="0.0 -3.552713678800501e-17 0.075" rpy="0.0 -0.0 0.0" />
-            <mass value="27.390760948486008" />
-            <inertia ixx="0.4793383165985121" iyy="0.47933831659848636" izz="0.8559612796401739" ixy="-3.3306690738754696e-16" iyz="3.3306690738754696e-16" ixz="0.0" />
+            <origin xyz="-3.552713678800501e-17 1.6653345369377347e-17 0.02623506611443311" rpy="0.0 -0.0 0.0" />
+            <mass value="1.3127916188565103" />
+            <inertia ixx="0.0033487094087884667" iyy="0.0033487094087883695" izz="0.00607267765883511" ixy="-1.3010426069826053e-18" iyz="-4.336808689942018e-19" ixz="-1.3877787807814457e-17" />
         </inertial>
         <visual name="f_wheel_l_visual">
-            <origin xyz="-0.4 -0.065 -0.425" rpy="1.5707963267948966 -0.0 0.0" />
+            <origin xyz="-0.15 -0.0025 -0.15937500000000002" rpy="1.5707963267948966 -0.0 0.0" />
             <geometry>
                 <mesh filename="package://amr_description/meshes/f_wheel_l.stl" scale="0.001 0.001 0.001" />
@@ -61,5 +61,5 @@
         </visual>
         <collision name="f_wheel_l_collision">
-            <origin xyz="-0.4 -0.065 -0.425" rpy="1.5707963267948966 -0.0 0.0" />
+            <origin xyz="-0.15 -0.0025 -0.15937500000000002" rpy="1.5707963267948966 -0.0 0.0" />
             <geometry>
                 <mesh filename="package://amr_description/meshes/f_wheel_l.stl" scale="0.001 0.001 0.001" />
@@ -69,10 +69,10 @@
     <link name="b_wheel_r">
         <inertial>
-            <origin xyz="0.0 3.552713678800501e-17 0.07500000000000007" rpy="0.0 -0.0 0.0" />
-            <mass value="27.390760948486008" />
-            <inertia ixx="0.47933831659850945" iyy="0.4793383165984846" izz="0.8559612796401739" ixy="3.3306690738754696e-16" iyz="-5.551115123125783e-16" ixz="-2.6645352591003757e-15" />
+            <origin xyz="1.7763568394002505e-17 -1.6653345369377347e-17 0.026235066114433145" rpy="0.0 -0.0 0.0" />
+            <mass value="1.31279161885651" />
+            <inertia ixx="0.0033487094087884667" iyy="0.0033487094087883695" izz="0.006072677658835093" ixy="-2.6020852139652106e-18" iyz="4.336808689942018e-19" ixz="6.938893903907228e-18" />
         </inertial>
         <visual name="b_wheel_r_visual">
-            <origin xyz="0.4 0.065 -0.425" rpy="-1.5707963267948966 -0.0 0.0" />
+            <origin xyz="0.15 0.0025 -0.15937500000000002" rpy="-1.5707963267948966 -0.0 0.0" />
             <geometry>
                 <mesh filename="package://amr_description/meshes/b_wheel_r.stl" scale="0.001 0.001 0.001" />
@@ -81,5 +81,5 @@
         </visual>
         <collision name="b_wheel_r_collision">
-            <origin xyz="0.4 0.065 -0.425" rpy="-1.5707963267948966 -0.0 0.0" />
+            <origin xyz="0.15 0.0025 -0.15937500000000002" rpy="-1.5707963267948966 -0.0 0.0" />
             <geometry>
                 <mesh filename="package://amr_description/meshes/b_wheel_r.stl" scale="0.001 0.001 0.001" />
@@ -89,10 +89,10 @@
     <link name="b_wheel_l">
         <inertial>
-            <origin xyz="0.0 -3.552713678800501e-17 0.075" rpy="0.0 -0.0 0.0" />
-            <mass value="27.390760948486008" />
-            <inertia ixx="0.4793383165985121" iyy="0.47933831659848636" izz="0.8559612796401739" ixy="-3.3306690738754696e-16" iyz="3.3306690738754696e-16" ixz="0.0" />
+            <origin xyz="1.7763568394002505e-17 2.997602166487923e-17 0.026235066114433145" rpy="0.0 -0.0 0.0" />
+            <mass value="1.31279161885651" />
+            <inertia ixx="0.0033487094087884736" iyy="0.0033487094087883557" izz="0.0060726776588351065" ixy="-1.0842021724855044e-19" iyz="2.2768245622195593e-18" ixz="0.0" />
         </inertial>
         <visual name="b_wheel_l_visual">
-            <origin xyz="0.4 -0.065 -0.425" rpy="1.5707963267948966 -0.0 0.0" />
+            <origin xyz="0.15 -0.0025 -0.15937500000000002" rpy="1.5707963267948966 -0.0 0.0" />
             <geometry>
                 <mesh filename="package://amr_description/meshes/b_wheel_l.stl" scale="0.001 0.001 0.001" />
@@ -101,5 +101,5 @@
         </visual>
         <collision name="b_wheel_l_collision">
-            <origin xyz="0.4 -0.065 -0.425" rpy="1.5707963267948966 -0.0 0.0" />
+            <origin xyz="0.15 -0.0025 -0.15937500000000002" rpy="1.5707963267948966 -0.0 0.0" />
             <geometry>
                 <mesh filename="package://amr_description/meshes/b_wheel_l.stl" scale="0.001 0.001 0.001" />
@@ -110,17 +110,16 @@
     <link name="camera_link">
         <inertial>
-            <origin xyz="0.00021147401675925437 1.1102230246251566e-18 0.05000000000000004" rpy="0.0 -0.0 0.0" />
-            <mass value="21.86537558266994" />
-            <inertia ixx="0.16402649642970402" iyy="0.03558843780421217" izz="0.16574154808891284" ixy="2.4125911295413974e-14" iyz="4.5693013817071915e-17" ixz="2.220446049250313e-16" />
+            <origin xyz="0.000784181248604554 -1.5090743243271368e-13 0.018750000000000037" rpy="0.0 -0.0 0.0" />
+            <mass value="0.03705472598311712" />
+            <inertia ixx="4.725459659822421e-05" iyy="1.3979668961784848e-05" izz="4.822081110235731e-05" ixy="8.065807004281012e-17" iyz="-8.66151594899114e-21" ixz="0.0" />
         </inertial>
         <visual name="camera_link_visual">
-            <origin xyz="-0.19166700333333336 1.1102230246251566e-18 -0.23500000000000001" rpy="0.0 -0.0 0.0" />
+            <origin xyz="-0.07187533333333333 1.1102230246251566e-18 -0.11" rpy="0.0 -0.0 0.0" />
             <geometry>
                 <mesh filename="package://amr_description/meshes/camera_link.stl" scale="0.001 0.001 0.001" />
             </geometry>
-            <material name="camera_link"/>
         </visual>
         <collision name="camera_link_collision">
-            <origin xyz="-0.19166700333333336 1.1102230246251566e-18 -0.23500000000000001" rpy="0.0 -0.0 0.0" />
+            <origin xyz="-0.07187533333333333 1.1102230246251566e-18 -0.11" rpy="0.0 -0.0 0.0" />
             <geometry>
                 <mesh filename="package://amr_description/meshes/camera_link.stl" scale="0.001 0.001 0.001" />
@@ -131,10 +130,10 @@
     <link name="lidar_link">
         <inertial>
-            <origin xyz="0.0 -1.8528073920390496e-17 0.04" rpy="0.0 -0.0 0.0" />
-            <mass value="30.826877913349836" />
-            <inertia ixx="0.13685849340280387" iyy="0.1368584934028112" izz="0.24083498369804202" ixy="1.8277205526828766e-16" iyz="3.1413946999236946e-17" ixz="0.0" />
+            <origin xyz="-3.335866296317086e-17 6.004559333370755e-17 0.015000000000000045" rpy="0.0 -0.0 0.0" />
+            <mass value="0.33441151294791577" />
+            <inertia ixx="0.00029211638344078025" iyy="0.00029211638344079304" izz="0.00048586532053086567" ixy="8.031975085032165e-19" iyz="-7.083755804160312e-19" ixz="9.091749575418355e-19" />
         </inertial>
         <visual name="lidar_link_visual">
-            <origin xyz="0.0 0.0 -0.185" rpy="3.141592653589793 -0.0 0.0" />
+            <origin xyz="0.0 0.0 -0.0475" rpy="3.141592653589793 -0.0 0.0" />
             <geometry>
                 <mesh filename="package://amr_description/meshes/lidar_link.stl" scale="0.001 0.001 0.001" />
@@ -143,5 +142,5 @@
         </visual>
         <collision name="lidar_link_collision">
-            <origin xyz="0.0 0.0 -0.185" rpy="3.141592653589793 -0.0 0.0" />
+            <origin xyz="0.0 0.0 -0.0475" rpy="3.141592653589793 -0.0 0.0" />
             <geometry>
                 <mesh filename="package://amr_description/meshes/lidar_link.stl" scale="0.001 0.001 0.001" />
@@ -151,5 +150,5 @@
 <!--Joints-->
     <joint name="f_wheel_r_revolute" type="continuous">
-        <origin xyz="0.4 -0.425 -0.065" rpy="1.5707963267948966 -0.0 0.0" />
+        <origin xyz="0.15 -0.15937500000000002 -0.0025" rpy="1.5707963267948966 -0.0 0.0" />
         <parent link="base_link" />
         <child link="f_wheel_r" />
@@ -158,5 +157,5 @@
     </joint>
     <joint name="f_wheel_l_revolute" type="continuous">
-        <origin xyz="0.4 0.425 -0.065" rpy="-1.5707963267948966 -0.0 0.0" />
+        <origin xyz="0.15 0.15937500000000002 -0.0025" rpy="-1.5707963267948966 -0.0 0.0" />
         <parent link="base_link" />
         <child link="f_wheel_l" />
@@ -165,5 +164,5 @@
     </joint>
     <joint name="b_wheel_l_revolute" type="continuous">
-        <origin xyz="-0.4 0.425 -0.065" rpy="-1.5707963267948966 -0.0 0.0" />
+        <origin xyz="-0.15 0.15937500000000002 -0.0025" rpy="-1.5707963267948966 -0.0 0.0" />
         <parent link="base_link" />
         <child link="b_wheel_l" />
@@ -172,5 +171,5 @@
     </joint>
     <joint name="b_wheel_r_revolute" type="continuous">
-        <origin xyz="-0.4 -0.425 -0.065" rpy="1.5707963267948966 -0.0 0.0" />
+        <origin xyz="-0.15 -0.15937500000000002 -0.0025" rpy="1.5707963267948966 -0.0 0.0" />
         <parent link="base_link" />
         <child link="b_wheel_r" />
@@ -179,5 +178,5 @@
     </joint>
     <joint name="camera_rotation" type="revolute">
-        <origin xyz="0.19166667 0.0 0.23500000000000001" rpy="0.0 -0.0 0.0" />
+        <origin xyz="0.07187500000000001 0.0 0.11" rpy="0.0 -0.0 0.0" />
         <parent link="base_link" />
         <child link="camera_link" />
@@ -186,5 +185,5 @@
     </joint>
     <joint name="lidar_rotation" type="continuous">
-        <origin xyz="0.0 0.0 -0.185" rpy="3.141592653589793 -0.0 0.0" />
+        <origin xyz="0.0 0.0 -0.0475" rpy="3.141592653589793 -0.0 0.0" />
         <parent link="base_link" />
         <child link="lidar_link" />
