Commit message: Editing the simulation

File: ros2_ws/install/amr_description/share/amr_description/urdf/amr.xacro (robot description, xacro)
@@ -1,246 +1 @@
-<?xml version='1.0' encoding='utf-8'?>
-<robot name="amr" xmlns:xacro="http://www.ros.org/wiki/xacro">
-  <!-- Include materials -->
-  <xacro:include filename="$(find amr_description)/urdf/materials.xacro"/>
-  <!-- Include gazebo -->
-  <xacro:include filename="$(find amr_description)/urdf/gazebo.xacro"/>
-<!--Base Link-->
-    <link name="base_link">
-        <inertial>
-            <origin xyz="-0.004351267108603693 -2.5010522091502847e-16 0.008281830778488642" rpy="0.0 0.0 0.0" />
-            <mass value="0.9360217886690454" />
-            <inertia ixx="0.009459041504582138" iyy="0.013956118845845198" izz="0.020474384137866695" ixy="5.096082182149493e-17" iyz="6.777214071700385e-17" ixz="0.00014505282040201085" />
-        </inertial>
-        <visual name="base_link_visual">
-            <origin xyz="0.0 0.0 0.0" rpy="0.0 0.0 0.0" />
-            <geometry>
-                <mesh filename="package://amr_description/meshes/base_link.stl" scale="0.001 0.001 0.001" />
-            </geometry>
-            <material name="base_link"/>
-        </visual>
-        <collision name="base_link_collision">
-            <origin xyz="0.0 0.0 0.0" rpy="0.0 0.0 0.0" />
-            <geometry>
-                <mesh filename="package://amr_description/meshes/base_link.stl" scale="0.001 0.001 0.001" />
-            </geometry>
-        </collision>
-    </link>
-<!--Wheels-->
-    <link name="f_wheel_r">
-        <inertial>
-            <origin xyz="-1.7763568394002505e-17 -4.440892098500626e-18 0.026235066114433145" rpy="0.0 -0.0 0.0" />
-            <mass value="1.3127916188565099" />
-            <inertia ixx="0.003348709408788453" iyy="0.0033487094087883557" izz="0.0060726776588351" ixy="-1.6263032587282567e-18" iyz="2.710505431213761e-18" ixz="0.0" />
-        </inertial>
-        <visual name="f_wheel_r_visual">
-            <origin xyz="-0.15 0.0025 -0.15937500000000002" rpy="-1.5707963267948966 -0.0 0.0" />
-            <geometry>
-                <mesh filename="package://amr_description/meshes/f_wheel_r.stl" scale="0.001 0.001 0.001" />
-            </geometry>
-            <material name="Wheels"/>
-        </visual>
-        <collision name="f_wheel_r_collision">
-            <origin xyz="-0.15 0.0025 -0.15937500000000002" rpy="-1.5707963267948966 -0.0 0.0" />
-            <geometry>
-                <mesh filename="package://amr_description/meshes/f_wheel_r.stl" scale="0.001 0.001 0.001" />
-            </geometry>
-        </collision>
-    </link>
-    <link name="f_wheel_l">
-        <inertial>
-            <origin xyz="-3.552713678800501e-17 1.6653345369377347e-17 0.02623506611443311" rpy="0.0 -0.0 0.0" />
-            <mass value="1.3127916188565103" />
-            <inertia ixx="0.0033487094087884667" iyy="0.0033487094087883695" izz="0.00607267765883511" ixy="-1.3010426069826053e-18" iyz="-4.336808689942018e-19" ixz="-1.3877787807814457e-17" />
-        </inertial>
-        <visual name="f_wheel_l_visual">
-            <origin xyz="-0.15 -0.0025 -0.15937500000000002" rpy="1.5707963267948966 -0.0 0.0" />
-            <geometry>
-                <mesh filename="package://amr_description/meshes/f_wheel_l.stl" scale="0.001 0.001 0.001" />
-            </geometry>
-            <material name="Wheels"/>
-        </visual>
-        <collision name="f_wheel_l_collision">
-            <origin xyz="-0.15 -0.0025 -0.15937500000000002" rpy="1.5707963267948966 -0.0 0.0" />
-            <geometry>
-                <mesh filename="package://amr_description/meshes/f_wheel_l.stl" scale="0.001 0.001 0.001" />
-            </geometry>
-        </collision>
-    </link>
-    <link name="b_wheel_r">
-        <inertial>
-            <origin xyz="1.7763568394002505e-17 -1.6653345369377347e-17 0.026235066114433145" rpy="0.0 -0.0 0.0" />
-            <mass value="1.31279161885651" />
-            <inertia ixx="0.0033487094087884667" iyy="0.0033487094087883695" izz="0.006072677658835093" ixy="-2.6020852139652106e-18" iyz="4.336808689942018e-19" ixz="6.938893903907228e-18" />
-        </inertial>
-        <visual name="b_wheel_r_visual">
-            <origin xyz="0.15 0.0025 -0.15937500000000002" rpy="-1.5707963267948966 -0.0 0.0" />
-            <geometry>
-                <mesh filename="package://amr_description/meshes/b_wheel_r.stl" scale="0.001 0.001 0.001" />
-            </geometry>
-            <material name="Wheels"/>
-        </visual>
-        <collision name="b_wheel_r_collision">
-            <origin xyz="0.15 0.0025 -0.15937500000000002" rpy="-1.5707963267948966 -0.0 0.0" />
-            <geometry>
-                <mesh filename="package://amr_description/meshes/b_wheel_r.stl" scale="0.001 0.001 0.001" />
-            </geometry>
-        </collision>
-    </link>
-    <link name="b_wheel_l">
-        <inertial>
-            <origin xyz="1.7763568394002505e-17 2.997602166487923e-17 0.026235066114433145" rpy="0.0 -0.0 0.0" />
-            <mass value="1.31279161885651" />
-            <inertia ixx="0.0033487094087884736" iyy="0.0033487094087883557" izz="0.0060726776588351065" ixy="-1.0842021724855044e-19" iyz="2.2768245622195593e-18" ixz="0.0" />
-        </inertial>
-        <visual name="b_wheel_l_visual">
-            <origin xyz="0.15 -0.0025 -0.15937500000000002" rpy="1.5707963267948966 -0.0 0.0" />
-            <geometry>
-                <mesh filename="package://amr_description/meshes/b_wheel_l.stl" scale="0.001 0.001 0.001" />
-            </geometry>
-            <material name="Wheels"/>
-        </visual>
-        <collision name="b_wheel_l_collision">
-            <origin xyz="0.15 -0.0025 -0.15937500000000002" rpy="1.5707963267948966 -0.0 0.0" />
-            <geometry>
-                <mesh filename="package://amr_description/meshes/b_wheel_l.stl" scale="0.001 0.001 0.001" />
-            </geometry>
-        </collision>
-    </link>
-<!--Camera link-->
-    <link name="camera_link">
-        <inertial>
-            <origin xyz="0.000784181248604554 -1.5090743243271368e-13 0.018750000000000037" rpy="0.0 -0.0 0.0" />
-            <mass value="0.03705472598311712" />
-            <inertia ixx="4.725459659822421e-05" iyy="1.3979668961784848e-05" izz="4.822081110235731e-05" ixy="8.065807004281012e-17" iyz="-8.66151594899114e-21" ixz="0.0" />
-        </inertial>
-        <visual name="camera_link_visual">
-            <origin xyz="-0.07187533333333333 1.1102230246251566e-18 -0.11" rpy="0.0 -0.0 0.0" />
-            <geometry>
-                <mesh filename="package://amr_description/meshes/camera_link.stl" scale="0.001 0.001 0.001" />
-            </geometry>
-        </visual>
-        <collision name="camera_link_collision">
-            <origin xyz="-0.07187533333333333 1.1102230246251566e-18 -0.11" rpy="0.0 -0.0 0.0" />
-            <geometry>
-                <mesh filename="package://amr_description/meshes/camera_link.stl" scale="0.001 0.001 0.001" />
-            </geometry>
-        </collision>
-    </link>
-<!--Lidar link-->
-    <link name="lidar_link">
-        <inertial>
-            <origin xyz="-3.335866296317086e-17 6.004559333370755e-17 0.015000000000000045" rpy="0.0 -0.0 0.0" />
-            <mass value="0.33441151294791577" />
-            <inertia ixx="0.00029211638344078025" iyy="0.00029211638344079304" izz="0.00048586532053086567" ixy="8.031975085032165e-19" iyz="-7.083755804160312e-19" ixz="9.091749575418355e-19" />
-        </inertial>
-        <visual name="lidar_link_visual">
-            <origin xyz="0.0 0.0 -0.0475" rpy="3.141592653589793 -0.0 0.0" />
-            <geometry>
-                <mesh filename="package://amr_description/meshes/lidar_link.stl" scale="0.001 0.001 0.001" />
-            </geometry>
-            <material name="lidar_link"/>
-        </visual>
-        <collision name="lidar_link_collision">
-            <origin xyz="0.0 0.0 -0.0475" rpy="3.141592653589793 -0.0 0.0" />
-            <geometry>
-                <mesh filename="package://amr_description/meshes/lidar_link.stl" scale="0.001 0.001 0.001" />
-            </geometry>
-        </collision>
-    </link>
-<!--Joints-->
-    <joint name="f_wheel_r_revolute" type="continuous">
-        <origin xyz="0.15 -0.15937500000000002 -0.0025" rpy="1.5707963267948966 -0.0 0.0" />
-        <parent link="base_link" />
-        <child link="f_wheel_r" />
-        <axis xyz="0.0 0.0 1.0" />
-        <dynamics damping="0.1" friction="0.1"/>
-    </joint>
-    <joint name="f_wheel_l_revolute" type="continuous">
-        <origin xyz="0.15 0.15937500000000002 -0.0025" rpy="-1.5707963267948966 -0.0 0.0" />
-        <parent link="base_link" />
-        <child link="f_wheel_l" />
-        <axis xyz="0.0 0.0 1.0" />
-        <dynamics damping="0.1" friction="0.1"/>
-    </joint>
-    <joint name="b_wheel_l_revolute" type="continuous">
-        <origin xyz="-0.15 0.15937500000000002 -0.0025" rpy="-1.5707963267948966 -0.0 0.0" />
-        <parent link="base_link" />
-        <child link="b_wheel_l" />
-        <axis xyz="0.0 0.0 1.0" />
-        <dynamics damping="0.1" friction="0.1"/>
-    </joint>
-    <joint name="b_wheel_r_revolute" type="continuous">
-        <origin xyz="-0.15 -0.15937500000000002 -0.0025" rpy="1.5707963267948966 -0.0 0.0" />
-        <parent link="base_link" />
-        <child link="b_wheel_r" />
-        <axis xyz="0.0 0.0 1.0" />
-        <dynamics damping="0.1" friction="0.1"/>
-    </joint>
-    <joint name="camera_rotation" type="revolute">
-        <origin xyz="0.07187500000000001 0.0 0.11" rpy="0.0 -0.0 0.0" />
-        <parent link="base_link" />
-        <child link="camera_link" />
-        <axis xyz="0.0 0.0 1.0" />
-        <limit lower="-1.5707963267948966" upper="1.5707963267948966" effort="100" velocity="1.0"/>
-    </joint>
-    <joint name="lidar_rotation" type="continuous">
-        <origin xyz="0.0 0.0 -0.0475" rpy="3.141592653589793 -0.0 0.0" />
-        <parent link="base_link" />
-        <child link="lidar_link" />
-        <axis xyz="0.0 0.0 1.0" />
-    </joint>
-    <!-- Camera Sensor Plugin -->
-        <gazebo reference="camera_link">
-            <sensor name="camera_sensor" type="camera">
-                <topic>camera/image_raw</topic>
-                <update_rate>30.0</update_rate>
-                <camera>
-                    <horizontal_fov>1.047</horizontal_fov>
-                    <image>
-                        <width>640</width>
-                        <height>480</height>
-                        <format>R8G8B8</format>
-                    </image>
-                    <clip>
-                        <near>0.1</near>
-                        <far>100.0</far>
-                    </clip>
-                </camera>
-                <plugin name="camera_controller" filename="libgazebo_ros_camera.so">
-                    <ros>
-                        <namespace>/camera</namespace>
-                    </ros>
-                    <frame_name>camera_link</frame_name>
-                </plugin>
-            </sensor>
-        </gazebo>
-    <!-- LiDAR Sensor Plugin -->
-        <gazebo reference="lidar_link">
-            <sensor name="lidar_sensor" type="ray">
-                <topic>scan</topic>
-                <update_rate>10.0</update_rate>
-                <ray>
-                    <scan>
-                        <horizontal>
-                            <samples>720</samples>
-                            <resolution>1</resolution>
-                            <min_angle>-3.14159</min_angle>
-                            <max_angle>3.14159</max_angle>
-                        </horizontal>
-                    </scan>
-                    <range>
-                        <min>0.12</min>
-                        <max>12.0</max>
-                        <resolution>0.01</resolution>
-                    </range>
-                </ray>
-                <plugin name="laser_controller" filename="libgazebo_ros_ray_sensor.so">
-                    <ros>
-                        <remapping>~/out:=scan</remapping>
-                    </ros>
-                    <output_type>sensor_msgs/LaserScan</output_type>
-                    <frame_name>lidar_link</frame_name>
-                </plugin>
-            </sensor>
-        </gazebo>
-</robot>
+/home/sam/amr-simulation/ros2_ws/src/amr_description/urdf/amr.xacro

File: ros2_ws/src/amr_description/urdf/gazebo.xacro (robot description, xacro)
@@ -3,5 +3,4 @@
     <!-- ================= BASE LINK ================= -->
     <gazebo reference="base_link">
-        <material>Gazebo/Orange</material>
         <mu1>1.0</mu1>
         <mu2>1.0</mu2>
@@ -9,7 +8,6 @@
         <kd>100.0</kd>
     </gazebo>
-    <!-- ================= RIGHT WHEEL 1 ================= -->
-    <gazebo reference="r_wheel_link_1">
-        <material>Gazebo/Black</material>
+    <!-- ================= front wheels ================= -->
+    <gazebo reference="f_wheel_r">
         <mu1>2.0</mu1>
         <mu2>2.0</mu2>
@@ -18,7 +16,5 @@
         <fdir1>1 0 0</fdir1>
     </gazebo>
-    <!-- ================= RIGHT WHEEL 2 ================= -->
-    <gazebo reference="r_wheel_link_2">
-        <material>Gazebo/Black</material>
+    <gazebo reference="f_wheel_l">
         <mu1>2.0</mu1>
         <mu2>2.0</mu2>
@@ -27,7 +23,6 @@
         <fdir1>1 0 0</fdir1>
     </gazebo>
-    <!-- ================= LEFT WHEEL 1 ================= -->
-    <gazebo reference="l_wheel_link_1">
-        <material>Gazebo/Black</material>
+    <!-- ================= back wheels ================= -->
+    <gazebo reference="b_wheel_r">
         <mu1>2.0</mu1>
         <mu2>2.0</mu2>
@@ -36,7 +31,5 @@
         <fdir1>1 0 0</fdir1>
     </gazebo>
-    <!-- ================= LEFT WHEEL 2 ================= -->
-    <gazebo reference="l_wheel_link_2">
-        <material>Gazebo/Black</material>
+    <gazebo reference="b_wheel_l">
         <mu1>2.0</mu1>
         <mu2>2.0</mu2>
@@ -62,10 +55,4 @@
                     </clip>
                 </camera>
-                <plugin name="camera_controller" filename="libgazebo_ros_camera.so">
-                    <ros>
-                        <namespace>/camera</namespace>
-                    </ros>
-                    <frame_name>camera_link</frame_name>
-                </plugin>
             </sensor>
         </gazebo>
@@ -90,11 +77,4 @@
                     </range>
                 </ray>
-                <plugin name="laser_controller" filename="libgazebo_ros_ray_sensor.so">
-                    <ros>
-                        <remapping>~/out:=scan</remapping>
-                    </ros>
-                    <output_type>sensor_msgs/LaserScan</output_type>
-                    <frame_name>lidar_link</frame_name>
-                </plugin>
             </sensor>
         </gazebo>
