Commit message: The amr successfully launched in RViz

File: ros2_ws/src/amr_description/urdf/amr.xacro (robot description, xacro)
@@ -5,4 +5,5 @@
   <!-- Include gazebo -->
   <xacro:include filename="$(find amr_description)/urdf/gazebo.xacro"/>
+    <link name="odom"/>
     <link name="base_link">
         <inertial>
@@ -16,4 +17,5 @@
                 <mesh filename="package://amr_description/meshes/base_link.stl" scale="0.001 0.001 0.001" />
             </geometry>
+            <material name="base_link"/>
         </visual>
         <collision name="base_link_collision">
@@ -35,4 +37,5 @@
                 <mesh filename="package://amr_description/meshes/f_wheel_r.stl" scale="0.001 0.001 0.001" />
             </geometry>
+            <material name="Wheels"/>
         </visual>
         <collision name="f_wheel_r_collision">
@@ -54,4 +57,5 @@
                 <mesh filename="package://amr_description/meshes/f_wheel_l.stl" scale="0.001 0.001 0.001" />
             </geometry>
+            <material name="Wheels"/>
         </visual>
         <collision name="f_wheel_l_collision">
@@ -73,4 +77,5 @@
                 <mesh filename="package://amr_description/meshes/b_wheel_r.stl" scale="0.001 0.001 0.001" />
             </geometry>
+            <material name="Wheels"/>
         </visual>
         <collision name="b_wheel_r_collision">
@@ -92,4 +97,5 @@
                 <mesh filename="package://amr_description/meshes/b_wheel_l.stl" scale="0.001 0.001 0.001" />
             </geometry>
+            <material name="Wheels"/>
         </visual>
         <collision name="b_wheel_l_collision">
@@ -112,4 +118,5 @@
                 <mesh filename="package://amr_description/meshes/camera_link.stl" scale="0.001 0.001 0.001" />
             </geometry>
+            <material name="camera_link"/>
         </visual>
         <collision name="camera_link_collision">
@@ -132,4 +139,5 @@
                 <mesh filename="package://amr_description/meshes/lidar_link.stl" scale="0.001 0.001 0.001" />
             </geometry>
+            <material name="lidar_link"/>
         </visual>
         <collision name="lidar_link_collision">
@@ -141,4 +149,9 @@
     </link>
 <!-- Joints -->
+    <joint name="odom_to_base_link" type="fixed">
+        <origin xyz="0.0 0.0 0.0" rpy="0.0 0.0 0.0" />
+        <parent link="odom" />
+        <child link="base_link" />
+    </joint>
     <joint name="base_link_f_wheel_r_revolute" type="continuous">
         <origin xyz="0.04 -0.0425 0.025" rpy="1.5707963267948966 -0.0 0.0" />

Commit message: Editing the simulaiton

File: ros2_ws/src/amr_description/urdf/amr.xacro (robot description, xacro)
@@ -154,5 +154,5 @@
         <child link="base_link" />
     </joint>
-    <joint name="base_link_f_wheel_r_revolute" type="continuous">
+    <joint name="f_wheel_r_revolute" type="continuous">
         <origin xyz="0.04 -0.0425 0.025" rpy="1.5707963267948966 -0.0 0.0" />
         <parent link="base_link" />
@@ -160,5 +160,5 @@
         <axis xyz="0.0 0.0 1.0" />
     </joint>
-    <joint name="base_link_f_wheel_l_revolute" type="continuous">
+    <joint name="f_wheel_l_revolute" type="continuous">
         <origin xyz="0.04 0.0425 0.025" rpy="-1.5707963267948966 -0.0 0.0" />
         <parent link="base_link" />
@@ -166,5 +166,5 @@
         <axis xyz="0.0 0.0 1.0" />
     </joint>
-    <joint name="base_link_b_wheel_l_revolute" type="continuous">
+    <joint name="b_wheel_l_revolute" type="continuous">
         <origin xyz="-0.04 0.0425 0.025" rpy="-1.5707963267948966 -0.0 0.0" />
         <parent link="base_link" />
@@ -172,5 +172,5 @@
         <axis xyz="0.0 0.0 1.0" />
     </joint>
-    <joint name="base_link_b_wheel_r_revolute" type="continuous">
+    <joint name="b_wheel_r_revolute" type="continuous">
         <origin xyz="-0.04 -0.0425 0.025" rpy="1.5707963267948966 -0.0 0.0" />
         <parent link="base_link" />
@@ -178,5 +178,5 @@
         <axis xyz="0.0 0.0 1.0" />
     </joint>
-    <joint name="base_link_camera_rotation" type="continuous">
+    <joint name="camera_rotation" type="continuous">
         <origin xyz="0.01916667 0.0 0.05" rpy="0.0 -0.0 0.0" />
         <parent link="base_link" />
@@ -184,5 +184,5 @@
         <axis xyz="0.0 0.0 1.0" />
     </joint>
-    <joint name="base_link_lidar_rotation" type="continuous">
+    <joint name="lidar_rotation" type="continuous">
         <origin xyz="-0.0275 0.0 0.06" rpy="0.0 -0.0 0.0" />
         <parent link="base_link" />

File: ros2_ws/src/amr_description/urdf/gazebo.xacro (robot description, xacro)
@@ -7,4 +7,5 @@
         <kp>1000000.0</kp>
         <kd>100.0</kd>
+        <collide_bitmask>0x00</collide_bitmask>
     </gazebo>
     <!-- ================= front wheels ================= -->
@@ -15,4 +16,5 @@
         <kd>100.0</kd>
         <fdir1>1 0 0</fdir1>
+        <collide_bitmask>0x00</collide_bitmask>
     </gazebo>
     <gazebo reference="f_wheel_l">
@@ -22,4 +24,5 @@
         <kd>100.0</kd>
         <fdir1>1 0 0</fdir1>
+        <collide_bitmask>0x00</collide_bitmask>
     </gazebo>
     <!-- ================= back wheels ================= -->
@@ -30,4 +33,5 @@
         <kd>100.0</kd>
         <fdir1>1 0 0</fdir1>
+        <collide_bitmask>0x00</collide_bitmask> // masks the collision of the wheel with the ground, allowing for smoother movement
     </gazebo>
     <gazebo reference="b_wheel_l">
@@ -37,4 +41,5 @@
         <kd>100.0</kd>
         <fdir1>1 0 0</fdir1>
+        <collide_bitmask>0x00</collide_bitmask>
     </gazebo>
     <!-- Camera Sensor Plugin -->

Commit message: Almost made the robot move

File: ros2_ws/src/amr_description/urdf/amr.xacro (robot description, xacro)
@@ -5,5 +5,4 @@
   <!-- Include gazebo -->
   <xacro:include filename="$(find amr_description)/urdf/gazebo.xacro"/>
-    <link name="odom"/>
     <link name="base_link">
         <inertial>
@@ -22,5 +21,5 @@
             <origin xyz="0.0 0.0 0.0" rpy="0.0 0.0 0.0" />
             <geometry>
-                <mesh filename="package://amr_description/meshes/base_link.stl" scale="0.001 0.001 0.001" />
+                <box size="0.10 0.03 0.010"/>
             </geometry>
         </collision>
@@ -42,5 +41,5 @@
             <origin xyz="-0.04 -0.025 -0.0425" rpy="-1.5707963267948966 -0.0 0.0" />
             <geometry>
-                <mesh filename="package://amr_description/meshes/f_wheel_r.stl" scale="0.001 0.001 0.001" />
+                <cylinder radius="0.05" length="0.015"/>
             </geometry>
         </collision>
@@ -62,5 +61,5 @@
             <origin xyz="-0.04 0.025 -0.0425" rpy="1.5707963267948966 -0.0 0.0" />
             <geometry>
-                <mesh filename="package://amr_description/meshes/f_wheel_l.stl" scale="0.001 0.001 0.001" />
+                <cylinder radius="0.05" length="0.015"/>
             </geometry>
         </collision>
@@ -82,5 +81,5 @@
             <origin xyz="0.04 -0.025 -0.0425" rpy="-1.5707963267948966 -0.0 0.0" />
             <geometry>
-                <mesh filename="package://amr_description/meshes/b_wheel_r.stl" scale="0.001 0.001 0.001" />
+                <cylinder radius="0.05" length="0.015"/>
             </geometry>
         </collision>
@@ -102,5 +101,5 @@
             <origin xyz="0.04 0.025 -0.0425" rpy="1.5707963267948966 -0.0 0.0" />
             <geometry>
-                <mesh filename="package://amr_description/meshes/b_wheel_l.stl" scale="0.001 0.001 0.001" />
+                <cylinder radius="0.05" length="0.015"/>
             </geometry>
         </collision>
@@ -123,5 +122,5 @@
             <origin xyz="-0.01916700333333333 1.1102230246251566e-18 -0.05" rpy="0.0 -0.0 0.0" />
             <geometry>
-                <mesh filename="package://amr_description/meshes/camera_link.stl" scale="0.001 0.001 0.001" />
+                <box size="0.011 0.030 0.010"/>
             </geometry>
         </collision>
@@ -144,14 +143,9 @@
             <origin xyz="0.0 4.996003610813204e-18 -0.037000000000000005" rpy="0.0 -0.0 0.0" />
             <geometry>
-                <mesh filename="package://amr_description/meshes/lidar_link.stl" scale="0.001 0.001 0.001" />
+                <cylinder radius="0.025" length="0.008"/>
             </geometry>
         </collision>
     </link>
 <!-- Joints -->
-    <joint name="odom_to_base_link" type="fixed">
-        <origin xyz="0.0 0.0 0.0" rpy="0.0 0.0 0.0" />
-        <parent link="odom" />
-        <child link="base_link" />
-    </joint>
     <joint name="f_wheel_r_revolute" type="continuous">
         <origin xyz="0.04 -0.0425 0.025" rpy="1.5707963267948966 -0.0 0.0" />

Commit message: Editing file

File: ros2_ws/src/amr_description/urdf/amr.xacro (robot description, xacro)
@@ -5,4 +5,5 @@
   <!-- Include gazebo -->
   <xacro:include filename="$(find amr_description)/urdf/gazebo.xacro"/>
+    <link name="base_footprint"/>
     <link name="base_link">
         <inertial>
@@ -148,4 +149,9 @@
     </link>
 <!-- Joints -->
+    <joint name="base_footprint_to_base_link" type="fixed">
+        <origin xyz="0.0 0.0 0.0" rpy="0.0 0.0 0.0" />
+        <parent link="base_footprint" />
+        <child link="base_link" />
+    </joint>
     <joint name="f_wheel_r_revolute" type="continuous">
         <origin xyz="0.04 -0.0425 0.025" rpy="1.5707963267948966 -0.0 0.0" />

File: ros2_ws/src/amr_description/urdf/gazebo.xacro (robot description, xacro)
@@ -7,5 +7,4 @@
         <kp>1000000.0</kp>
         <kd>100.0</kd>
-        <collide_bitmask>0x00</collide_bitmask>
     </gazebo>
     <!-- ================= front wheels ================= -->
@@ -16,5 +15,4 @@
         <kd>100.0</kd>
         <fdir1>1 0 0</fdir1>
-        <collide_bitmask>0x00</collide_bitmask>
     </gazebo>
     <gazebo reference="f_wheel_l">
@@ -24,5 +22,4 @@
         <kd>100.0</kd>
         <fdir1>1 0 0</fdir1>
-        <collide_bitmask>0x00</collide_bitmask>
     </gazebo>
     <!-- ================= back wheels ================= -->
@@ -33,5 +30,4 @@
         <kd>100.0</kd>
         <fdir1>1 0 0</fdir1>
-        <collide_bitmask>0x00</collide_bitmask> // masks the collision of the wheel with the ground, allowing for smoother movement
     </gazebo>
     <gazebo reference="b_wheel_l">
@@ -41,5 +37,4 @@
         <kd>100.0</kd>
         <fdir1>1 0 0</fdir1>
-        <collide_bitmask>0x00</collide_bitmask>
     </gazebo>
     <!-- Camera Sensor Plugin -->

Commit message: Editing Simulation

File: ros2_ws/src/amr_description/urdf/amr.xacro (robot description, xacro)
@@ -15,5 +15,5 @@
             <origin xyz="0.0 0.0 0.0" rpy="0.0 0.0 0.0" />
             <geometry>
-                <mesh filename="package://amr_description/meshes/base_link.stl" scale="0.001 0.001 0.001" />
+                <mesh filename="file://$(find amr_description)/meshes/base_link.stl" scale="0.001 0.001 0.001" />
             </geometry>
             <material name="base_link"/>
@@ -35,5 +35,5 @@
             <origin xyz="-0.04 -0.025 -0.0425" rpy="-1.5707963267948966 -0.0 0.0" />
             <geometry>
-                <mesh filename="package://amr_description/meshes/f_wheel_r.stl" scale="0.001 0.001 0.001" />
+                <mesh filename="file://$(find amr_description)/meshes/f_wheel_r.stl" scale="0.001 0.001 0.001" />
             </geometry>
             <material name="Wheels"/>
@@ -55,5 +55,5 @@
             <origin xyz="-0.04 0.025 -0.0425" rpy="1.5707963267948966 -0.0 0.0" />
             <geometry>
-                <mesh filename="package://amr_description/meshes/f_wheel_l.stl" scale="0.001 0.001 0.001" />
+                <mesh filename="file://$(find amr_description)/meshes/f_wheel_l.stl" scale="0.001 0.001 0.001" />
             </geometry>
             <material name="Wheels"/>
@@ -75,5 +75,5 @@
             <origin xyz="0.04 -0.025 -0.0425" rpy="-1.5707963267948966 -0.0 0.0" />
             <geometry>
-                <mesh filename="package://amr_description/meshes/b_wheel_r.stl" scale="0.001 0.001 0.001" />
+                <mesh filename="file://$(find amr_description)/meshes/b_wheel_r.stl" scale="0.001 0.001 0.001" />
             </geometry>
             <material name="Wheels"/>
@@ -95,5 +95,5 @@
             <origin xyz="0.04 0.025 -0.0425" rpy="1.5707963267948966 -0.0 0.0" />
             <geometry>
-                <mesh filename="package://amr_description/meshes/b_wheel_l.stl" scale="0.001 0.001 0.001" />
+                <mesh filename="file://$(find amr_description)/meshes/b_wheel_l.stl" scale="0.001 0.001 0.001" />
             </geometry>
             <material name="Wheels"/>
@@ -116,5 +116,5 @@
             <origin xyz="-0.01916700333333333 1.1102230246251566e-18 -0.05" rpy="0.0 -0.0 0.0" />
             <geometry>
-                <mesh filename="package://amr_description/meshes/camera_link.stl" scale="0.001 0.001 0.001" />
+                <mesh filename="file://$(find amr_description)/meshes/camera_link.stl" scale="0.001 0.001 0.001" />
             </geometry>
             <material name="camera_link"/>
@@ -137,5 +137,5 @@
             <origin xyz="0.0 4.996003610813204e-18 -0.037000000000000005" rpy="0.0 -0.0 0.0" />
             <geometry>
-                <mesh filename="package://amr_description/meshes/lidar_link.stl" scale="0.001 0.001 0.001" />
+                <mesh filename="file://$(find amr_description)/meshes/lidar_link.stl" scale="0.001 0.001 0.001" />
             </geometry>
             <material name="lidar_link"/>

File: ros2_ws/src/amr_description/urdf/gazebo.xacro (robot description, xacro)
@@ -41,5 +41,5 @@
         <gazebo reference="camera_link">
             <sensor name="camera_sensor" type="camera">
-                <topic>camera/image_raw</topic>
+                <topic>camera/image</topic>
                 <update_rate>30.0</update_rate>
                 <camera>
